Commit message: added RGB camera sim

File: bumperbot_description/urdf/bumperbot.urdf.xacro (robot description, xacro)
@@ -206,4 +206,28 @@
     <axis xyz="0 0 0" />
   </joint>
+  <link name="rgb_camera">
+    <mass value="0.0001" />
+    <inertia ixx="0.001" ixy="0.001" ixz="0.001"
+             iyy="0.001" iyz="0.001"
+             izz="0.001" />
+    <visual>
+      <origin rpy="0.0 0.0 0.0" xyz="0.0 0.0 0.0"/>
+      <geometry>
+        <mesh filename="package://bumperbot_description/meshes/pi_camera.STL"/>
+      </geometry>
+      <material name="green"/>
+    </visual>
+    <collision>
+      <origin rpy="0.0 0.0 0.0" xyz="0.0 0.0 0.0"/>
+      <geometry>
+        <mesh filename="package://bumperbot_description/meshes/pi_camera.STL"/>
+      </geometry>
+    </collision>
+  </link>
+  <joint name ="rgb_camera_joint" type="fixed">
+    <parent link="base_link"/>
+    <child link = "rgb_camera"/>
+    <origin xyz="0.078 0.0 0.07" rpy="0.0 -0.35 0.0"/>
+  </joint>
   <material name="blue">
     <color rgba="0 0 1 1"/>
@@ -218,3 +242,6 @@
     <color rgba="0.3 0.3 0.3 1"/>
   </material>
+  <material name="green">
+    <color rgba="0 1 0 1"/>
+  </material>
 </robot>

File: bumperbot_description/urdf/bumperbot_gazebo.xacro (robot description, xacro)
@@ -143,3 +143,29 @@
     </sensor>
   </gazebo>
+  <!-- RGB Camera -->
+  <gazebo reference="rgb_camera">
+    <sensor name="camera" type="camera">
+      <always_on>true</always_on>
+      <update_rate>30.0</update_rate>
+      <visualize>true</visualize>
+      <topic>/image_raw</topic>
+      <gz_frame_id>/rgb_camera</gz_frame_id>
+      <camera name="camera">
+        <horizontal_fov>1.21126</horizontal_fov>
+        <image>
+          <width>2304</width>
+          <height>1296</height>
+          <format>R8G8B8</format>
+        </image>
+        <distortion>
+          <k1>0.0</k1>
+          <k2>0.0</k2>
+          <k3>0.0</k3>
+          <p1>0.0</p1>
+          <p2>0.0</p2>
+          <center>0.5 0.5</center>
+        </distortion>
+      </camera>
+    </sensor>
+  </gazebo>
 </robot>

Commit message: added depth camera

File: bumperbot_description/urdf/bumperbot.urdf.xacro (robot description, xacro)
@@ -5,8 +5,12 @@
   <!-- Load Simulated or Real Hardware Interfaces -->
   <xacro:arg name="is_sim" default="true"/>
+  <xacro:arg name="camera_model" default="realsense_d435"/>
+  <xacro:property name="camera_model" value="$(arg camera_model)" />
   <!-- Include Gazebo Parameters -->
   <xacro:include filename="$(find bumperbot_description)/urdf/bumperbot_gazebo.xacro" />
   <!-- Include ros2_control Plugins -->
   <xacro:include filename="$(find bumperbot_description)/urdf/bumperbot_ros2_control.xacro" />
+  <!-- Include Realsense Description -->
+  <xacro:include filename="$(find realsense2_description)/urdf/_d435.urdf.xacro"/>
   <link name="base_footprint"/>
   <link name="base_link">
@@ -206,28 +210,35 @@
     <axis xyz="0 0 0" />
   </joint>
-  <link name="rgb_camera">
-    <mass value="0.0001" />
-    <inertia ixx="0.001" ixy="0.001" ixz="0.001"
-             iyy="0.001" iyz="0.001"
-             izz="0.001" />
-    <visual>
-      <origin rpy="0.0 0.0 0.0" xyz="0.0 0.0 0.0"/>
-      <geometry>
-        <mesh filename="package://bumperbot_description/meshes/pi_camera.STL"/>
-      </geometry>
-      <material name="green"/>
-    </visual>
-    <collision>
-      <origin rpy="0.0 0.0 0.0" xyz="0.0 0.0 0.0"/>
-      <geometry>
-        <mesh filename="package://bumperbot_description/meshes/pi_camera.STL"/>
-      </geometry>
-    </collision>
-  </link>
-  <joint name ="rgb_camera_joint" type="fixed">
-    <parent link="base_link"/>
-    <child link = "rgb_camera"/>
-    <origin xyz="0.078 0.0 0.07" rpy="0.0 -0.35 0.0"/>
-  </joint>
+  <xacro:if value="${camera_model == 'pi_camera'}">
+    <link name="rgb_camera">
+      <mass value="0.0001" />
+      <inertia ixx="0.001" ixy="0.001" ixz="0.001"
+              iyy="0.001" iyz="0.001"
+              izz="0.001" />
+      <visual>
+        <origin rpy="0.0 0.0 0.0" xyz="0.0 0.0 0.0"/>
+        <geometry>
+          <mesh filename="package://bumperbot_description/meshes/pi_camera.STL"/>
+        </geometry>
+        <material name="green"/>
+      </visual>
+      <collision>
+        <origin rpy="0.0 0.0 0.0" xyz="0.0 0.0 0.0"/>
+        <geometry>
+          <mesh filename="package://bumperbot_description/meshes/pi_camera.STL"/>
+        </geometry>
+      </collision>
+    </link>
+    <joint name ="camera_joint" type="fixed">
+      <parent link="base_link"/>
+      <child link = "rgb_camera"/>
+      <origin xyz="0.078 0.0 0.07" rpy="0.0 -0.35 0.0"/>
+    </joint>
+  </xacro:if>
+  <xacro:if value="${camera_model == 'realsense_d435'}">
+    <xacro:sensor_d435 name="rgbd_camera" parent="base_link" use_nominal_extrinsics="$(arg is_sim)">
+      <origin xyz="0.07 0.0 0.08" rpy="0.0 0.0 0.0"/>
+    </xacro:sensor_d435>
+  </xacro:if>
   <material name="blue">
     <color rgba="0 0 1 1"/>

File: bumperbot_description/urdf/bumperbot_gazebo.xacro (robot description, xacro)
@@ -144,28 +144,84 @@
   </gazebo>
   <!-- RGB Camera -->
-  <gazebo reference="rgb_camera">
-    <sensor name="camera" type="camera">
-      <always_on>true</always_on>
-      <update_rate>30.0</update_rate>
-      <visualize>true</visualize>
-      <topic>/image_raw</topic>
-      <gz_frame_id>/rgb_camera</gz_frame_id>
-      <camera name="camera">
-        <horizontal_fov>1.21126</horizontal_fov>
-        <image>
-          <width>2304</width>
-          <height>1296</height>
-          <format>R8G8B8</format>
-        </image>
-        <distortion>
-          <k1>0.0</k1>
-          <k2>0.0</k2>
-          <k3>0.0</k3>
-          <p1>0.0</p1>
-          <p2>0.0</p2>
-          <center>0.5 0.5</center>
-        </distortion>
-      </camera>
-    </sensor>
-  </gazebo>
+  <xacro:if value="${camera_model == 'pi_camera'}">
+    <gazebo reference="rgb_camera">
+      <sensor name="camera" type="camera">
+        <always_on>true</always_on>
+        <update_rate>30.0</update_rate>
+        <visualize>true</visualize>
+        <topic>/image_raw</topic>
+        <gz_frame_id>/rgb_camera</gz_frame_id>
+        <camera name="camera">
+          <horizontal_fov>1.21126</horizontal_fov>
+          <image>
+            <width>2304</width>
+            <height>1296</height>
+            <format>R8G8B8</format>
+          </image>
+          <distortion>
+            <k1>0.0</k1>
+            <k2>0.0</k2>
+            <k3>0.0</k3>
+            <p1>0.0</p1>
+            <p2>0.0</p2>
+            <center>0.5 0.5</center>
+          </distortion>
+        </camera>
+      </sensor>
+    </gazebo>
+  </xacro:if>
+  <!-- RGBD Camera -->
+  <xacro:if value="${camera_model == 'realsense_d435'}">
+    <gazebo reference="rgbd_camera_link">
+      <sensor name="d435_color" type="camera">
+				<always_on>1</always_on>
+				<update_rate>30</update_rate>
+				<visualize>1</visualize>
+				<pose>0 0.0175 0.5125 0 -0 0</pose>
+				<topic>/rgbd_camera/image_raw</topic>
+        <gz_frame_id>rgbd_camera_link</gz_frame_id>
+				<camera name="d435">
+					<horizontal_fov>1.21126</horizontal_fov>
+					<image>
+						<width>640</width>
+						<height>480</height>
+						<format>RGB_INT8</format>
+					</image>
+					<clip>
+						<near>0.1</near>
+						<far>100</far>
+					</clip>
+					<noise>
+						<type>gaussian</type>
+						<mean>0</mean>
+						<stddev>0.007</stddev>
+					</noise>
+				</camera>
+			</sensor>
+      <sensor name="d435_depth" type="depth_camera">
+				<always_on>1</always_on>
+				<update_rate>90</update_rate>
+				<visualize>0</visualize>
+				<topic>/rgbd_camera/depth</topic>
+        <gz_frame_id>rgbd_camera_link</gz_frame_id>
+				<pose>0 0.0175 0.5125 0 -0 0</pose>
+				<camera name="d435">
+					<horizontal_fov>1.48702</horizontal_fov>
+					<image>
+						<width>1280</width>
+						<height>720</height>
+					</image>
+					<clip>
+						<near>0.1</near>
+						<far>100</far>
+					</clip>
+					<noise>
+						<type>gaussian</type>
+						<mean>0</mean>
+						<stddev>0.1</stddev>
+					</noise>
+				</camera>
+			</sensor>
+    </gazebo>
+  </xacro:if>
 </robot>

Commit message: added image undistrort

File: bumperbot_description/urdf/bumperbot.urdf.xacro (robot description, xacro)
@@ -5,12 +5,8 @@
   <!-- Load Simulated or Real Hardware Interfaces -->
   <xacro:arg name="is_sim" default="true"/>
-  <xacro:arg name="camera_model" default="realsense_d435"/>
-  <xacro:property name="camera_model" value="$(arg camera_model)" />
   <!-- Include Gazebo Parameters -->
   <xacro:include filename="$(find bumperbot_description)/urdf/bumperbot_gazebo.xacro" />
   <!-- Include ros2_control Plugins -->
   <xacro:include filename="$(find bumperbot_description)/urdf/bumperbot_ros2_control.xacro" />
-  <!-- Include Realsense Description -->
-  <xacro:include filename="$(find realsense2_description)/urdf/_d435.urdf.xacro"/>
   <link name="base_footprint"/>
   <link name="base_link">

File: bumperbot_description/urdf/bumperbot_gazebo.xacro (robot description, xacro)
@@ -159,7 +159,8 @@
           <format>R8G8B8</format>
         </image>
+        <!-- Simulate Barrel distorsion -->
         <distortion>
-          <k1>0.0</k1>
-          <k2>0.0</k2>
+          <k1>-0.01</k1>
+          <k2>0.005</k2>
           <k3>0.0</k3>
           <p1>0.0</p1>
@@ -185,7 +186,8 @@
           <format>R8G8B8</format>
         </image>
+        <!-- Simulate Pincushion distorsion -->
         <distortion>
-          <k1>0.0</k1>
-          <k2>0.0</k2>
+          <k1>0.01</k1>
+          <k2>0.005</k2>
           <k3>0.0</k3>
           <p1>0.0</p1>

Commit message: using image_pipeline

File: bumperbot_description/urdf/bumperbot.urdf.xacro (robot description, xacro)
@@ -236,4 +236,10 @@
     <origin xyz="0.0 -0.06 0.0" rpy="0.0 0.0 0.0"/>
   </joint>
+  <link name="right_camera_optical_link"/>
+  <joint name="right_camera_optical_joint" type="fixed">
+    <parent link="right_camera_link"/>
+    <child link="right_camera_optical_link"/>
+    <origin xyz="0 0 0" rpy="-1.571 0 -1.571"/>
+  </joint>
   <link name="left_camera_link"/>
   <joint name ="left_camera_joint" type="fixed">
@@ -242,4 +248,10 @@
     <origin xyz="0.0 0.0 0.0" rpy="0.0 0.0 0.0"/>
   </joint>
+  <link name="left_camera_optical_link"/>
+  <joint name="left_camera_optical_joint" type="fixed">
+    <parent link="left_camera_link"/>
+    <child link="left_camera_optical_link"/>
+    <origin xyz="0 0 0" rpy="-1.571 0 -1.571"/>
+  </joint>
   <material name="blue">
     <color rgba="0 0 1 1"/>

File: bumperbot_description/urdf/bumperbot_gazebo.xacro (robot description, xacro)
@@ -150,5 +150,5 @@
       <visualize>true</visualize>
       <topic>/left_camera/image_raw</topic>
-      <gz_frame_id>left_camera_link</gz_frame_id>
+      <gz_frame_id>left_camera_optical_link</gz_frame_id>
       <camera name="left_camera">
         <horizontal_fov>1.27409</horizontal_fov>
@@ -177,5 +177,5 @@
       <visualize>true</visualize>
       <topic>/right_camera/image_raw</topic>
-      <gz_frame_id>right_camera_link</gz_frame_id>
+      <gz_frame_id>right_camera_optical_link</gz_frame_id>
       <camera name="right_camera">
         <horizontal_fov>1.27409</horizontal_fov>
